File: Attiny828/DecoderconBEC/Decodificador de ppm.sch (EAGLE design)
At the start: 21 parts, among them U1 ATTINY828-AURTQFP32_9X9_MCH-M, U2 AP63205WU-7SOIC_05WU-7_DIO-M

Commit message: Add files via upload
Se agrego capcitor de entrada del regulador un canal menos y mejor perfil
Parts:
- removed SV1, SV5: (no value), con-lstb:MA03-1
- added C3: (no value), rcl:C-EUC0805
- added TP7, TP8, TP9: TPTP19SQ, testpad:TPTP19SQ
- TP5, TP6: value TPB1,27 -> TPTP19SQ; device testpad:TPB1,27 -> testpad:TPTP19SQ
Connections:
- removed net N$10: SV5.3, U1.(PCINT3/ADC3)_PA3
- net +5V: now also TP8.TP; no longer SV1.2, SV5.2
- net GND: now also C3.1, TP9.TP; no longer SV1.1, SV5.1
- net N$3: now also TP7.TP; no longer SV1.3
- net V+: now also C3.2
